File: meth.sch (KiCad schematic (older format))
At the start: 36 parts, among them IC1 ATMEGA32-P, J1 ETHERNET, P1 GPIO1, P2 GPIO2, P3 ISP, P4 UART, P5 SD CARD, P6 POWER, SW1 DUAL_SWITCH_INV, SW2 DUAL_SWITCH_INV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

Commit message: newer kicad
Connections:
- wire segments 128 -> 140
Other:
- moved on the sheet: C1, C2, C3, C6, C7, C8, P6, R6
Changed lines of the file:
@@
 LIBS:memory
 LIBS:xilinx
-LIBS:special
 LIBS:microcontrollers
 LIBS:dsp
@@
 LIBS:valves
 LIBS:meth
-EELAYER 24 0
+LIBS:meth-cache
+EELAYER 25 0
 EELAYER END
 $Descr A4 11693 8268
@@
 L C C1
 U 1 1 550425F7
-P 5600 4150
-F 0 "C1" V 5650 4200 40  0000 L CNN
-F 1 "10pF" V 5550 3950 40  0000 L CNN
-F 2 "" H 5638 4000 30  0000 C CNN
-F 3 "" H 5600 4150 60  0000 C CNN
-	1    5600 4150
+P 5650 4150
+F 0 "C1" V 5700 4200 40  0000 L CNN
+F 1 "10pF" V 5600 3950 40  0000 L CNN
+F 2 "" H 5688 4000 30  0000 C CNN
+F 3 "" H 5650 4150 60  0000 C CNN
+	1    5650 4150
 	0    1    1    0
 $EndComp
@@
 L C C2
 U 1 1 5504260B
-P 5600 4750
-F 0 "C2" V 5650 4800 40  0000 L CNN
-F 1 "10pF" V 5550 4550 40  0000 L CNN
-F 2 "" H 5638 4600 30  0000 C CNN
-F 3 "" H 5600 4750 60  0000 C CNN
-	1    5600 4750
+P 5650 4750
+F 0 "C2" V 5700 4800 40  0000 L CNN
+F 1 "10pF" V 5600 4550 40  0000 L CNN
+F 2 "" H 5688 4600 30  0000 C CNN
+F 3 "" H 5650 4750 60  0000 C CNN
+	1    5650 4750
 	0    1    1    0
 $EndComp
@@
 L GND #PWR04
 U 1 1 55042648
-P 5200 4550
-F 0 "#PWR04" H 5200 4550 30  0001 C CNN
-F 1 "GND" H 5200 4480 30  0001 C CNN
-F 2 "" H 5200 4550 60  0000 C CNN
-F 3 "" H 5200 4550 60  0000 C CNN
-	1    5200 4550
+P 5350 4550
+F 0 "#PWR04" H 5350 4550 30  0001 C CNN
+F 1 "GND" H 5350 4480 30  0001 C CNN
+F 2 "" H 5350 4550 60  0000 C CNN
+F 3 "" H 5350 4550 60  0000 C CNN
+	1    5350 4550
 	1    0    0    -1
 $EndComp
@@
 L R R6
 U 1 1 55042687
-P 5750 3850
-F 0 "R6" V 5830 3850 40  0000 C CNN
-F 1 "2.32k" V 5757 3851 40  0000 C CNN
-F 2 "" V 5680 3850 30  0000 C CNN
-F 3 "" H 5750 3850 30  0000 C CNN
-	1    5750 3850
+P 5800 3850
+F 0 "R6" V 5880 3850 40  0000 C CNN
+F 1 "2.32k" V 5807 3851 40  0000 C CNN
+F 2 "" V 5730 3850 30  0000 C CNN
+F 3 "" H 5800 3850 30  0000 C CNN
+	1    5800 3850
 	0    1    1    0
 $EndComp
@@
 L C C3
 U 1 1 5504269B
-P 5800 3650
-F 0 "C3" V 5850 3700 40  0000 L CNN
-F 1 "10uF" V 5750 3450 40  0000 L CNN
-F 2 "" H 5838 3500 30  0000 C CNN
-F 3 "" H 5800 3650 60  0000 C CNN
-	1    5800 3650
+P 5700 3650
+F 0 "C3" V 5750 3700 40  0000 L CNN
+F 1 "10uF" V 5650 3450 40  0000 L CNN
+F 2 "" H 5738 3500 30  0000 C CNN
+F 3 "" H 5700 3650 60  0000 C CNN
+	1    5700 3650
 	0    1    1    0
 $EndComp
@@
 L C C7
 U 1 1 55047C48
-P 10300 4950
-F 0 "C7" H 10300 5050 40  0000 L CNN
-F 1 "10uF" H 10306 4865 40  0000 L CNN
-F 2 "" H 10338 4800 30  0000 C CNN
-F 3 "" H 10300 4950 60  0000 C CNN
-	1    10300 4950
+P 10300 4900
+F 0 "C7" H 10300 5000 40  0000 L CNN
+F 1 "10uF" H 10306 4815 40  0000 L CNN
+F 2 "" H 10338 4750 30  0000 C CNN
+F 3 "" H 10300 4900 60  0000 C CNN
+	1    10300 4900
 	1    0    0    -1
 $EndComp
@@
 L C C6
 U 1 1 55047C5C
-P 9500 4950
-F 0 "C6" H 9500 5050 40  0000 L CNN
-F 1 "10uF" H 9506 4865 40  0000 L CNN
-F 2 "" H 9538 4800 30  0000 C CNN
-F 3 "" H 9500 4950 60  0000 C CNN
-	1    9500 4950
+P 9500 4900
+F 0 "C6" H 9500 5000 40  0000 L CNN
+F 1 "10uF" H 9506 4815 40  0000 L CNN
+F 2 "" H 9538 4750 30  0000 C CNN
+F 3 "" H 9500 4900 60  0000 C CNN
+	1    9500 4900
 	1    0    0    -1
 $EndComp
@@
 L GND #PWR020
 U 1 1 55047DBC
-P 9900 5400
-F 0 "#PWR020" H 9900 5400 30  0001 C CNN
-F 1 "GND" H 9900 5330 30  0001 C CNN
-F 2 "" H 9900 5400 60  0000 C CNN
-F 3 "" H 9900 5400 60  0000 C CNN
-	1    9900 5400
+P 9900 5300
+F 0 "#PWR020" H 9900 5300 30  0001 C CNN
+F 1 "GND" H 9900 5230 30  0001 C CNN
+F 2 "" H 9900 5300 60  0000 C CNN
+F 3 "" H 9900 5300 60  0000 C CNN
+	1    9900 5300
 	1    0    0    -1
 $EndComp
@@
 L CONN_2 P6
 U 1 1 55047F1E
-P 8850 4950
-F 0 "P6" V 8800 4950 40  0000 C CNN
-F 1 "POWER" V 8900 4950 40  0000 C CNN
-F 2 "" H 8850 4950 60  0000 C CNN
-F 3 "" H 8850 4950 60  0000 C CNN
-	1    8850 4950
+P 8850 4900
+F 0 "P6" V 8800 4900 40  0000 C CNN
+F 1 "POWER" V 8900 4900 40  0000 C CNN
+F 2 "" H 8850 4900 60  0000 C CNN
+F 3 "" H 8850 4900 60  0000 C CNN
+	1    8850 4900
 	-1   0    0    1
 $EndComp
@@
 L C C8
 U 1 1 5505CEC9
-P 1950 1350
-F 0 "C8" V 1900 1450 40  0000 L CNN
-F 1 "0.1uF" V 2100 1300 40  0000 L CNN
-F 2 "" H 1988 1200 30  0000 C CNN
-F 3 "" H 1950 1350 60  0000 C CNN
-	1    1950 1350
+P 1900 1350
+F 0 "C8" V 1850 1450 40  0000 L CNN
+F 1 "0.1uF" V 1750 1250 40  0000 L CNN
+F 2 "" H 1938 1200 30  0000 C CNN
+F 3 "" H 1900 1350 60  0000 C CNN
+	1    1900 1350
 	0    1    1    0
 $EndComp
@@
 L GND #PWR023
 U 1 1 5505CF87
-P 2150 1450
-F 0 "#PWR023" H 2150 1450 30  0001 C CNN
-F 1 "GND" H 2150 1380 30  0001 C CNN
-F 2 "" H 2150 1450 60  0000 C CNN
-F 3 "" H 2150 1450 60  0000 C CNN
-	1    2150 1450
+P 2050 1450
+F 0 "#PWR023" H 2050 1450 30  0001 C CNN
+F 1 "GND" H 2050 1380 30  0001 C CNN
+F 2 "" H 2050 1450 60  0000 C CNN
+F 3 "" H 2050 1450 60  0000 C CNN
+	1    2050 1450
 	1    0    0    -1
 $EndComp
@@
 L PWR_FLAG #FLG026
 U 1 1 550B60DA
-P 9900 5300
-F 0 "#FLG026" H 9900 5395 30  0001 C CNN
-F 1 "PWR_FLAG" H 9900 5480 30  0000 C CNN
-F 2 "" H 9900 5300 60  0000 C CNN
-F 3 "" H 9900 5300 60  0000 C CNN
-	1    9900 5300
+P 9900 5200
+F 0 "#FLG026" H 9900 5295 30  0001 C CNN
+F 1 "PWR_FLAG" H 9900 5380 30  0000 C CNN
+F 2 "" H 9900 5200 60  0000 C CNN
+F 3 "" H 9900 5200 60  0000 C CNN
+	1    9900 5200
 	0    1    1    0
 $EndComp
@@
 	8800 2650 9400 2650
 Wire Wire Line
-	8800 3150 8800 2650
+	8800 2650 8800 3200
 Wire Wire Line
 	8550 3150 8800 3150
@@
 Connection ~ 8600 3150
 Wire Wire Line
-	8600 3050 8600 3250
+	8600 2950 8600 3350
 Connection ~ 7950 2950
 Wire Wire Line
@@
 	7950 2350 9400 2350
 Wire Wire Line
-	7950 2250 7950 2450
+	7950 2150 7950 2550
 Wire Wire Line
 	9100 4000 9100 2950
@@
 Connection ~ 9300 3050
 Wire Wire Line
-	5400 4150 5400 4750
-Wire Wire Line
-	5200 3650 5200 4550
-Wire Wire Line
-	5200 4400 5400 4400
-Connection ~ 5400 4400
+	5500 4150 5500 4750
+Wire Wire Line
+	5350 3650 5350 4550
+Connection ~ 5500 4400
 Wire Wire Line
 	6000 4250 6000 4750
 Wire Wire Line
-	5500 3850 5200 3850
-Connection ~ 5200 4400
-Wire Wire Line
-	5200 3650 5600 3650
-Connection ~ 5200 3850
+	5650 3850 5350 3850
+Connection ~ 5350 4400
+Connection ~ 5350 3850
 Wire Wire Line
 	6550 2150 7050 2150
@@
 	5900 2950 5900 3350
 Wire Wire Line
-	8100 4000 9100 4000
-Wire Wire Line
-	9200 4100 8500 4100
-Wire Wire Line
-	7600 4100 8000 4100
+	8000 4000 9100 4000
+Wire Wire Line
+	9200 4100 8400 4100
+Wire Wire Line
+	7600 4100 8100 4100
 Wire Wire Line
 	5700 3050 6000 3050
@@
 	2600 3350 5800 3350
 Wire Wire Line
-	2600 3250 3950 3250
+	2600 3250 4050 3250
 Wire Wire Line
 	2600 3050 3950 3050
@@
 	5900 3350 6000 3350
 Wire Wire Line
-	4450 3250 5700 3250
+	4350 3250 5700 3250
 Wire Wire Line
 	2600 3150 6000 3150
@@
 	5200 2400 5200 2600
 Wire Wire Line
-	7950 1750 7950 1550
+	7950 1550 7950 1850
 Connection ~ 7950 1550
 Connection ~ 4800 3250
@@
 	4600 4650 4600 4750
 Wire Wire Line
-	9350 5150 10300 5150
-Wire Wire Line
-	9200 5050 9350 5050
-Wire Wire Line
-	9350 5050 9350 5150
-Wire Wire Line
-	9200 4850 9350 4850
-Wire Wire Line
-	9350 4850 9350 4750
+	9350 5050 10300 5050
+Wire Wire Line
+	9200 5000 9350 5000
+Wire Wire Line
+	9200 4800 9350 4800
 Wire Wire Line
 	9350 4750 9500 4750
@@
 Wire Wire Line
 	10400 4750 10400 4650
-Wire Wire Line
-	9900 5050 9900 5400
 Connection ~ 3400 2350
 Connection ~ 3400 2250
@@
 	7800 1550 8350 1550
 Wire Wire Line
-	2150 1450 2150 1350
+	2050 1450 2050 1350
 Wire Wire Line
 	1750 1350 1450 1350
@@
 	8150 1650 8150 1450
 Wire Wire Line
-	8150 2350 8150 2250
+	8150 2250 8150 2400
 Connection ~ 8150 2350
 Wire Wire Line
@@
 	3050 5600 3050 6000
 Wire Wire Line
-	4200 6000 3550 6000
-Wire Wire Line
-	3550 5250 4200 5250
-Wire Wire Line
-	4200 6250 3750 6250
+	3450 6000 4200 6000
+Wire Wire Line
+	3450 5250 4200 5250
+Wire Wire Line
+	3650 6250 4200 6250
 Connection ~ 4200 6000
 Wire Wire Line
-	4200 6550 3750 6550
+	3650 6550 4200 6550
 Connection ~ 4200 6250
 Connection ~ 4200 6550
 Connection ~ 10300 4750
 Connection ~ 9500 4750
-Connection ~ 9500 5150
+Connection ~ 9500 5050
 Text Notes 9400 4450 0    60   ~ 0
 Power Supply
-Connection ~ 9900 5150
+Connection ~ 9900 5050
 Connection ~ 1750 1350
-Connection ~ 9900 5300
+Connection ~ 9900 5200
+Wire Wire Line
+	5950 3850 6000 3850
+Wire Wire Line
+	5350 4400 5500 4400
+Wire Wire Line
+	5850 3650 6000 3650
+Wire Wire Line
+	5350 3650 5550 3650
+Wire Wire Line
+	7600 4000 7700 4000
+Wire Wire Line
+	9900 5300 9900 5050
+Wire Wire Line
+	9350 4800 9350 4750
+Wire Wire Line
+	9350 5000 9350 5050
+Wire Wire Line
+	7950 2850 7950 2950
+Wire Wire Line
+	8150 2750 8150 2700
+Wire Wire Line
+	8600 2650 8600 2550
+Wire Wire Line
+	8600 3750 8600 3650
+Connection ~ 8800 3150
+Wire Wire Line
+	8800 3550 8800 3500
+Wire Wire Line
+	3350 6250 3250 6250
+Wire Wire Line
+	3250 6550 3350 6550
+Wire Wire Line
+	3050 6000 3150 6000
+Wire Wire Line
+	3050 5250 3150 5250
 $EndSCHEMATC
