File: meth.kicad_pcb (KiCad board)
At the start: 2 copper layers, 94 x 85.1 mm, 36 parts, among them IC1 ATMEGA32-P, J1 ETHERNET, P1 GPIO1, P2 GPIO2, P3 ISP, P4 UART, P5 SD CARD, P6 POWER, SW1 DUAL_SWITCH_INV, SW2 DUAL_SWITCH_INV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

Commit message: Reroute
Routing:
- net GND: track 682.3 -> 716.9 mm
- net +3.3V: track 287.6 -> 304.4 mm
- net Net-(C4-Pad1): track 57.6 -> 69.4 mm
- net Net-(IC1-Pad3): track 72.7 -> 80.1 mm
- net Net-(IC1-Pad4): track 78.9 -> 82.3 mm
- net Net-(IC1-Pad16): track 62.0 -> 59.1 mm
- net Net-(IC1-Pad17): track 49.6 -> 52.5 mm
- net Net-(C2-Pad1): track 30.5 -> 33.0 mm
- net Net-(P5-Pad1): track 60.2 -> 62.7 mm
- net Net-(R8-Pad2): track 46.0 -> 43.6 mm
- net Net-(J1-Pad4): track 36.4 -> 38.8 mm
- net Net-(C5-Pad1): track 31.8 -> 33.3 mm
- net Net-(J1-Pad1): track 30.4 -> 31.8 mm
- net Net-(C6-Pad1): track 29.6 -> 30.6 mm
- net Net-(IC1-Pad6): track 73.3 -> 74.3 mm
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Other:
- net class Default: clearance 0.254 -> 0.2; trace_width 0.254 -> 0.3
- rule trace_clearance: 0.254 -> 0.2
- board text added: "v1.1"
- board text removed: "v1.0"

Commit message: Optimize
Routing:
- net Net-(P5-Pad1): track 62.7 -> 80.6 mm
- net GND: track 716.9 -> 727.5 mm
- net Net-(IC1-Pad8): track 87.6 -> 94.5 mm
- net Net-(IC1-Pad6): track 74.3 -> 80.7 mm
- net Net-(IC1-Pad4): track 82.3 -> 88.1 mm
- net Net-(IC1-Pad16): track 59.1 -> 62.4 mm
- net Net-(J1-Pad1): track 31.8 -> 35.0 mm
- net Net-(IC1-Pad17): track 52.5 -> 53.8 mm
- net Net-(J1-Pad3): track 41.2 -> 42.5 mm

Commit message: Fill
Routing:
- net GND: track 727.5 -> 742.8 mm
- net +3.3V: track 304.4 -> 315.9 mm
- net Net-(IC1-Pad8): track 94.5 -> 100.7 mm
- net Net-(J1-Pad6): track 37.9 -> 42.2 mm
- net Net-(C5-Pad1): track 33.3 -> 30.1 mm
- net Net-(IC1-Pad17): track 53.8 -> 56.9 mm
- net Net-(C1-Pad1): track 30.0 -> 33.1 mm
- net Net-(IC1-Pad7): track 21.7 -> 24.4 mm
- net Net-(C4-Pad1): track 69.4 -> 70.5 mm
- net Net-(IC1-Pad16): track 62.4 -> 63.4 mm
- net Net-(C2-Pad1): track 33.0 -> 33.9 mm
- added copper zone on B.Cu, net GND

Commit message: Some rerouting
Routing:
- net GND: track 742.8 -> 752.8 mm
- net Net-(D2-Pad2): track 16.0 -> 20.1 mm
- net Net-(D1-Pad1): track 80.9 -> 84.4 mm
- net Net-(IC1-Pad3): track 80.1 -> 83.3 mm
- net +3.3V: track 315.9 -> 318.9 mm
- net Net-(IC1-Pad8): track 100.7 -> 103.1 mm
- net Net-(IC1-Pad4): track 88.1 -> 89.3 mm
- net Net-(IC1-Pad2): track 16.8 -> 17.6 mm

Commit message: Fixups
Routing:
- net GND: track 752.8 -> 765.3 mm
- net +3.3V: track 318.9 -> 322.5 mm
